Commit message: code cleanup

File: autobot_description/urdf/autobot.urdf (robot description, URDF)
Before this commit: robot autobot, 6 links, 5 joints
Links:
- added link imu_link, mass 1e-5; collision box size=0.025 0.025 0.0025; visual box size=0.025 0.025 0.0025
Joints:
- added joint imu_joint: type fixed, parent base_link, child imu_link, origin xyz=0.075 0 0.1025 rpy=0 0 0, axis 0 0 0

Commit message: finally installed xacro

File: autobot_description/urdf/autobot.urdf (robot description, URDF)
Before this commit: robot autobot, 7 links, 6 joints
Links:
- link base_link: geometry collision mesh filename=$(find autobot_gazebo)/meshes/base_link.STL; visual mesh filename=$(find autobot_gazebo)/meshes/base_link.STL
- link left_back_link: geometry collision mesh filename=$(find autobot_gazebo)/meshes/left_back_link.STL; visual mesh filename=$(find autobot_gazebo)/meshes/left_back_link.STL
- link left_front_link: geometry collision mesh filename=$(find autobot_gazebo)/meshes/left_front_link.STL; visual mesh filename=$(find autobot_gazebo)/meshes/left_front_link.STL
- link lidar_link: geometry collision mesh filename=$(find autobot_gazebo)/meshes/lidar_link.STL; visual mesh filename=$(find autobot_gazebo)/meshes/lidar_link.STL
- link right_back_link: geometry collision mesh filename=$(find autobot_gazebo)/meshes/right_back_link.STL; visual mesh filename=$(find autobot_gazebo)/meshes/right_back_link.STL
- link right_front_link: geometry collision mesh filename=$(find autobot_gazebo)/meshes/right_front_link.STL; visual mesh filename=$(find autobot_gazebo)/meshes/right_front_link.STL

Commit message: added new gazebo world

File: autobot_description/urdf/autobot.urdf (robot description, URDF)
Before this commit: robot autobot, 7 links, 6 joints
Links:
- added link base_footprint
- link base_link: geometry collision mesh filename=$(find autobot_gazebo)/models/autobot/meshes/base_link.STL; visual mesh filename=$(find autobot_gazebo)/models/autobot/meshes/base_link.STL
- link left_back_link: geometry collision mesh filename=$(find autobot_gazebo)/models/autobot/meshes/left_back_link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; visual mesh filename=$(find autobot_gazebo)/models/autobot/meshes/left_back_link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
- link left_front_link: geometry collision mesh filename=$(find autobot_gazebo)/models/autobot/meshes/left_front_lin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; visual mesh filename=$(find autobot_gazebo)/models/autobot/meshes/left_front_lin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
- link lidar_link: geometry collision mesh filename=$(find autobot_gazebo)/models/autobot/meshes/lidar_link.STL; visual mesh filename=$(find autobot_gazebo)/models/autobot/meshes/lidar_link.STL
- link right_back_link: geometry collision mesh filename=$(find autobot_gazebo)/models/autobot/meshes/right_back_lin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; visual mesh filename=$(find autobot_gazebo)/models/autobot/meshes/right_back_lin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
- link right_front_link: geometry collision mesh filename=$(find autobot_gazebo)/models/autobot/meshes/right_front_li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; visual mesh filename=$(find autobot_gazebo)/models/autobot/meshes/right_front_li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
Joints:
- added joint base_joint: type fixed, parent base_link, child base_footprint, origin xyz=0.0 0.0 -0.0518795 rpy=0 0 0

Commit message: camera attachment

File: autobot_description/urdf/autobot.urdf (robot description, URDF)
Before this commit: robot autobot, 8 links, 7 joints
Links:
- added link camera_link, mass 1e-5; collision box size=0.03 0.03 0.03; visual box size=0.03 0.03 0.03
- added link camera_link_optical
Joints:
- added joint camera_joint: type fixed, parent base_link, child camera_link, origin xyz=0.123 0 0.035 rpy=0 0.1 0, axis 1 0 0
- added joint camera_optical_joint: type fixed, parent camera_link, child camera_link_optical, origin xyz=0 0 0 rpy=${-pi/2} 0 ${-pi/2}

File: autobot_description/urdf/plugins.xacro (robot description, xacro)
@@ -130,4 +130,26 @@
       <material>Gazebo/Black</material>
   </gazebo>
+  <gazebo reference="camera_link">
+    <sensor name="camera" type="camera">
+      <pose> 0 0 0 0 0 0 </pose>
+      <visualize>true</visualize>
+      <update_rate>10</update_rate>
+      <camera>
+        <horizontal_fov>1.089</horizontal_fov>
+        <image>
+          <format>R8G8B8</format>
+          <width>640</width>
+          <height>480</height>
+        </image>
+        <clip>
+          <near>0.05</near>
+          <far>8.0</far>
+        </clip>
+      </camera>
+      <plugin name="camera_controller" filename="libgazebo_ros_camera.so">
+        <frame_name>camera_link_optical</frame_name>
+      </plugin>
+    </sensor>
+  </gazebo>
   <gazebo reference="base_link">
       <material>Gazebo/White</material>
@@ -145,3 +167,6 @@
       <material>Gazebo/Grey</material>
   </gazebo>
+  <gazebo reference="camera_link">
+      <material>Gazebo/Red</material>
+  </gazebo>
 </launch>
